Commit message: removed build deps.

File: turtlebot3_ws/src/auto_park/description/turtlebot3_burger.urdf.xacro (robot description, xacro)
@@ -13,5 +13,5 @@
       <origin xyz="-0.032 0 0.0" rpy="0 0 0"/>
       <geometry>
-        <mesh filename="file:///home/ubuntu/project/turtlebot3_ws/src/auto_park/description/burger_base.stl" scale="0.001 0.001 0.001"/>
+        <mesh filename="file:///home/ubuntu/auto_parking/turtlebot3_ws/src/auto_park/description/burger_base.stl" scale="0.001 0.001 0.001"/>
       </geometry>
       <material name="light_black"/>
@@ -41,5 +41,5 @@
       <origin xyz="0 0 0" rpy="1.57 0 0"/>
       <geometry>
-        <mesh filename="file:///home/ubuntu/project/turtlebot3_ws/src/auto_park/description/left_tire.stl" scale="0.001 0.001 0.001"/>
+        <mesh filename="file:///home/ubuntu/auto_parking/turtlebot3_ws/src/auto_park/description/left_tire.stl" scale="0.001 0.001 0.001"/>
       </geometry>
       <material name="dark"/>
@@ -69,5 +69,5 @@
       <origin xyz="0 0 0" rpy="1.57 0 0"/>
       <geometry>
-        <mesh filename="file:///home/ubuntu/project/turtlebot3_ws/src/auto_park/description/right_tire.stl" scale="0.001 0.001 0.001"/>
+        <mesh filename="file:///home/ubuntu/auto_parking/turtlebot3_ws/src/auto_park/description/right_tire.stl" scale="0.001 0.001 0.001"/>
       </geometry>
       <material name="dark"/>
@@ -122,5 +122,5 @@
       <origin xyz="0 0 0.0" rpy="0 0 0"/>
       <geometry>
-        <mesh filename="file:///home/ubuntu/project/turtlebot3_ws/src/auto_park/description/lds.stl" scale="0.001 0.001 0.001"/>
+        <mesh filename="file:///home/ubuntu/auto_parking/turtlebot3_ws/src/auto_park/description/lds.stl" scale="0.001 0.001 0.001"/>
       </geometry>
       <material name="dark"/>
@@ -357,5 +357,5 @@
   <gazebo>
     <plugin name="gazebo_ros2_control" filename="libgazebo_ros2_control.so">
-      <parameters>/home/ubuntu/project/turtlebot3_ws/src/auto_park/config/controllers.yaml</parameters>
+      <parameters>/home/ubuntu/auto_parking/turtlebot3_ws/src/auto_park/config/controllers.yaml</parameters>
     </plugin>
   </gazebo>

Commit message: tracking

File: turtlebot3_ws/src/auto_park/description/turtlebot3_burger.urdf.xacro (robot description, xacro)
@@ -163,5 +163,5 @@
     <parent link="base_link"/>
     <child link="camera_link"/>
-    <origin xyz="-0.089 0 0.1144" rpy="0 0.18 ${pi}"/>
+    <origin xyz="0.029 0 0.1147" rpy="0 0.18 0"/>
   </joint>
   <link name="camera_link">
@@ -357,9 +357,9 @@
     <plugin name="gazebo_ros2_control" filename="libgazebo_ros2_control.so">
       <parameters>/home/ubuntu/auto_parking/turtlebot3_ws/src/auto_park/config/controllers.yaml</parameters>
-      <!--  <odometry_frame>odom</odometry_frame>
+      <odometry_frame>odom</odometry_frame>
       <robot_base_frame>base_link</robot_base_frame>
       <publish_odom>true</publish_odom>
       <publish_odom_tf>true</publish_odom_tf>
-      <publish_wheel_tf>true</publish_wheel_tf> -->
+      <publish_wheel_tf>true</publish_wheel_tf>
    </plugin>
   </gazebo>
