Commit message: car2

File: car_ws/src/auto_park2/description/prius.urdf.xacro (robot description, xacro)
@@ -1,4 +1,5 @@
 <?xml version="1.0"?>
 <robot name="prius" xmlns:xacro="http://ros.org/wiki/xacro">
+  <xacro:include filename="common_properties.xacro"/>
   <link name="base_footprint">
     <inertial>
@@ -10,5 +11,5 @@
     <parent link="base_footprint"/>
     <child link="base_link"/>
-    <origin xyz="1.45 0 0" rpy="0 0 1.57"/>
+    <origin xyz="1.45 0 0.31265" rpy="0 0 1.57"/>
     <axis xyz="1 0 0"/>
   </joint>
@@ -16,7 +17,7 @@
   <link name="base_link">
     <visual>
-      <origin xyz="0 1.45 -0.3" rpy="0 0 0"/>
-      <geometry>
-        <mesh filename="file:///home/ubuntu/auto_parking/car_ws/src/auto_park2/description/hybrid_body.obj" scale="0.01 0.01 0.01"/>
+      <origin xyz="0 1.42 -0.3" rpy="0 0 0"/>
+      <geometry>
+        <mesh filename="file:///home/andrew/auto_parking/car_ws/src/auto_park2/description/hybrid_body.obj" scale="0.01 0.01 0.01"/>
       </geometry>
       <material name="light_black"/>
@@ -28,18 +29,67 @@
       </geometry>
     </collision>
-    <inertial>
-      <mass value="1356.0"/>
+    <collision name="front_bumper">
+      <origin xyz="0.0 -2.0 0.458488" rpy="0.0 0 0"/>
+      <geometry>
+        <box size="1.337282 0.48 0.566691"/>
+      </geometry>
+    </collision>
+    <collision name="hood">
+      <origin xyz="0.0 -1.900842 0.676305" rpy="0.341247 0 0"/>
+      <geometry>
+        <box size="1.597968 0.493107 0.265468"/>
+      </geometry>
+    </collision>
+    <collision name="windshield">
+      <origin xyz="0.0 -0.875105 1.032268" rpy="0.335476 0 0"/>
+      <geometry>
+        <box size="1.168381 1.654253 0.272347"/>
+      </geometry>
+    </collision>
+    <collision name="top_front">
+      <origin xyz="0.0 0.161236 1.386042" rpy="0.135030 0 0"/>
+      <geometry>
+        <box size="1.279154 0.625988 0.171868"/>
+      </geometry>
+    </collision>
+    <collision name="top_rear">
+      <origin xyz="0.0 0.817696 1.360069" rpy="-0.068997 0 0"/>
+      <geometry>
+        <box size="1.285130 0.771189 0.226557"/>
+      </geometry>
+    </collision>
+    <collision name="rear_window">
+      <origin xyz="0.0 1.640531 1.175126" rpy="-0.262017 0 0"/>
+      <geometry>
+        <box size="1.267845 1.116344 0.244286"/>
+      </geometry>
+    </collision>
+    <collision name="trunk">
+      <origin xyz="0.0 1.637059 0.888180" rpy="0.0 0 0"/>
+      <geometry>
+        <box size="1.788064 1.138988 0.482746"/>
+      </geometry>
+    </collision>
+    <collision name="back_bumper">
+      <origin xyz="0.0 2.054454 0.577870" rpy="0.0 0 0"/>
+      <geometry>
+        <box size="1.781650 0.512093 0.581427"/>
+      </geometry>
+    </collision>
+    <inertial>
+      <mass value="100.0"/>
       <origin xyz="0 0 0.48" rpy="0 0 1.5708"/>
-      <inertia ixx="2581.13354740" ixy="0.0" ixz="0.0"
-               iyy="591.30846112" iyz="0.0"
-               izz="2681.95008628"/>
-    </inertial>
-  </link>
-  <!-- left_wheel -->
+      <inertia ixx="190.264166667" ixy="0.0" ixz="0.0"
+               iyy="197.576666667" iyz="0.0"
+               izz="44.3141666667"/>
+    </inertial>
+  </link>
+  <!-- front left_wheel -->
   <joint name="wheel_left_joint" type="continuous">
-    <parent link="base_link"/>
+    <parent link="fl_axle"/>
     <child link="wheel_left_link"/>
-    <origin xyz="0.0 0.88 0.0" rpy="0 0 0"/>
+    <origin xyz="0.0 0.0 0.0" rpy="0 0 0"/>
     <axis xyz="1 0 0"/>
+    <limit effort="1000.0" velocity="10.0" lower="-0.8727" upper="0.8727"/>
   </joint>
   <link name="wheel_left_link">
@@ -47,5 +97,5 @@
       <origin xyz="0 0 0" rpy="0 0 0"/>
       <geometry>
-        <mesh filename="file:///home/ubuntu/auto_parking/car_ws/src/auto_park2/description/wheel.obj" scale="0.01 0.01 0.01"/>
+        <mesh filename="file:///home/andrew/auto_parking/car_ws/src/auto_park2/description/wheel.obj" scale="0.01 0.01 0.01"/>
       </geometry>
     </visual>
@@ -61,10 +111,25 @@
     </collision>
   </link>
-  <!-- right_wheel -->
+  <!-- front left axle -->
+  <link name="fl_axle">
+    <inertial>
+      <mass value="1"/>
+      <origin xyz="0 0 0"/>
+      <inertia ixx="0.004" ixy="0.0" ixz="0.0" iyy="0.004" iyz="0.0" izz="0.004"/>
+    </inertial>
+  </link>
+  <joint name="front_left_steer_joint" type="fixed">
+    <parent link="base_link"/>
+    <child link="fl_axle"/>
+    <origin xyz="0.8 0 0" rpy="0 0 0"/>
+    <axis xyz="0 0 1"/>
+  </joint>
+  <!-- front right_wheel -->
   <joint name="wheel_right_joint" type="continuous">
-    <parent link="base_link"/>
-    <child link="wheel_left_link"/>
-    <origin xyz="0.0 -0.88 0.0" rpy="0 0 0"/>
+    <parent link="fr_axle"/>
+    <child link="wheel_right_link"/>
+    <origin xyz="0.0 0.0 0.0" rpy="0 0 0"/>
     <axis xyz="1 0 0"/>
+    <limit effort="1000.0" velocity="10.0" lower="-0.8727" upper="0.8727"/>
   </joint>
   <link name="wheel_right_link">
@@ -72,5 +137,5 @@
       <origin xyz="0 0 0" rpy="0 0 0"/>
       <geometry>
-        <mesh filename="file:///home/ubuntu/auto_parking/car_ws/src/auto_park2/description/wheel.obj" scale="0.01 0.01 0.01"/>
+        <mesh filename="file:///home/andrew/auto_parking/car_ws/src/auto_park2/description/wheel.obj" scale="0.01 0.01 0.01"/>
       </geometry>
     </visual>
@@ -86,3 +151,416 @@
     </collision>
   </link>
+  <!-- front right axle -->
+  <link name="fr_axle">
+    <inertial>
+      <mass value="1"/>
+      <origin xyz="0 0 0"/>
+      <inertia ixx="0.004" ixy="0.0" ixz="0.0" iyy="0.004" iyz="0.0" izz="0.004"/>
+    </inertial>
+  </link>
+  <joint name="front_right_steer_joint" type="fixed">
+    <parent link="base_link"/>
+    <child link="fr_axle"/>
+    <origin xyz="-0.8 0 0" rpy="0 0 0"/>
+    <axis xyz="0 0 1"/>
+  </joint>
+  <!-- rear left_wheel -->
+  <joint name="rear_wheel_left_joint" type="continuous">
+    <parent link="base_footprint"/>
+    <child link="rear_wheel_left_link"/>
+    <origin xyz="-1.41 0.8 0.31265" rpy="0 0 ${pi/2}"/>
+    <axis xyz="1 0 0"/>
+  </joint>
+  <link name="rear_wheel_left_link">
+    <visual>
+      <origin xyz="0 0 0" rpy="0 0 0"/>
+      <geometry>
+        <mesh filename="file:///home/andrew/auto_parking/car_ws/src/auto_park2/description/wheel.obj" scale="0.01 0.01 0.01"/>
+      </geometry>
+    </visual>
+    <inertial>
+      <mass value="11"/>
+      <origin xyz="0 0 0"/>
+      <inertia ixx="0.58631238" ixy="0.0" ixz="0.0" iyy="0.33552910" iyz="0.0" izz="0.33552910"/>
+    </inertial>
+    <collision name="rear_left_wheel_collision">
+      <geometry>
+        <sphere radius="0.31265"/>
+      </geometry>
+    </collision>
+  </link>
+  <!-- rear right_wheel -->
+  <joint name="rear_wheel_right_joint" type="continuous">
+    <parent link="base_footprint"/>
+    <child link="rear_wheel_right_link"/>
+    <origin xyz="-1.41 -0.8 0.31265" rpy="0 0 ${pi/2}"/>
+    <axis xyz="1 0 0"/>
+  </joint>
+  <link name="rear_wheel_right_link">
+    <visual>
+      <origin xyz="0 0 0" rpy="0 0 0"/>
+      <geometry>
+        <mesh filename="file:///home/andrew/auto_parking/car_ws/src/auto_park2/description/wheel.obj" scale="0.01 0.01 0.01"/>
+      </geometry>
+    </visual>
+    <inertial>
+      <mass value="11"/>
+      <origin xyz="0 0 0"/>
+      <inertia ixx="0.58631238" ixy="0.0" ixz="0.0" iyy="0.33552910" iyz="0.0" izz="0.33552910"/>
+    </inertial>
+    <collision name="rear_right_wheel_collision">
+      <geometry>
+        <sphere radius="0.31265"/>
+      </geometry>
+    </collision>
+  </link>
+  <!-- imu -->
+  <joint name="imu_joint" type="fixed">
+    <parent link="base_link"/>
+    <child link="imu_link"/>
+    <origin xyz="0 0 0" rpy="0 0 0"/>
+  </joint>
+  <link name="imu_link"/>
+  <!-- lasers -->
+  <link name="base_scan">
+    <inertial>
+      <mass value="1"/>
+      <inertia ixx="0.001" ixy="0.0" ixz="0.0" iyy="0.001" iyz="0.0" izz="0.001"/>
+    </inertial>
+  </link>
+  <joint name="scan_joint" type="fixed">
+    <parent link="base_link"/>
+    <child link="base_scan"/>
+    <origin xyz="0 0.5 1.125" rpy="0 0 -1.5707"/>
+  </joint>
+  <!-- front camera -->
+  <link name="front_camera_link">
+    <inertial>
+      <mass value="1"/>
+      <inertia ixx="0.001" ixy="0.0" ixz="0.0" iyy="0.001" iyz="0.0" izz="0.001"/>
+    </inertial>
+    <visual>
+      <origin xyz="0 0 0" rpy="0 0 0"/>
+      <geometry>
+        <box size="0.010 0.03 0.03"/>
+      </geometry>
+      <material name="red"/>
+    </visual>
+  </link>
+  <joint name="front_camera_joint" type="fixed">
+    <parent link="base_link"/>
+    <child link="front_camera_link"/>
+    <origin xyz="0 -0.63 0.5" rpy="0 0.05 -1.5707"/>
+  </joint>
+  <link name="front_camera_link_optical">
+    <inertial>
+      <mass value="1"/>
+      <inertia ixx="0.001" ixy="0.0" ixz="0.0" iyy="0.001" iyz="0.0" izz="0.001"/>
+    </inertial>
+  </link>
+  <joint name="front_camera_optical_joint" type="fixed">
+    <origin xyz="0 0 0" rpy="-1.5707 0 -1.5707"/>
+    <parent link="front_camera_link"/>
+    <child link="front_camera_link_optical"/>
+  </joint>
+  <!-- back camera -->
+  <link name="back_camera_link">
+    <inertial>
+      <mass value="1"/>
+      <inertia ixx="0.001" ixy="0.0" ixz="0.0" iyy="0.001" iyz="0.0" izz="0.001"/>
+    </inertial>
+    <visual>
+      <origin xyz="0 0 0" rpy="0 0 0"/>
+      <geometry>
+        <box size="0.010 0.03 0.03"/>
+      </geometry>
+      <material name="red"/>
+    </visual>
+  </link>
+  <joint name="back_camera_joint" type="fixed">
+    <parent link="base_link"/>
+    <child link="back_camera_link"/>
+    <origin xyz="0 3.67 0.64" rpy="0 0.05 1.5707"/>
+  </joint>
+  <link name="back_camera_link_optical">
+    <inertial>
+      <mass value="1"/>
+      <inertia ixx="0.001" ixy="0.0" ixz="0.0" iyy="0.001" iyz="0.0" izz="0.001"/>
+    </inertial>
+  </link>
+  <joint name="back_camera_optical_joint" type="fixed">
+    <origin xyz="0 0 0" rpy="-1.5707 0 -1.5707"/>
+    <parent link="back_camera_link"/>
+    <child link="back_camera_link_optical"/>
+  </joint>
+  <!-- left camera -->
+  <link name="left_camera_link">
+    <inertial>
+      <mass value="1"/>
+      <inertia ixx="0.001" ixy="0.0" ixz="0.0" iyy="0.001" iyz="0.0" izz="0.001"/>
+    </inertial>
+    <visual>
+      <origin xyz="0 0 0" rpy="0 0 0"/>
+      <geometry>
+        <box size="0.010 0.03 0.03"/>
+      </geometry>
+      <material name="red"/>
+    </visual>
+  </link>
+  <joint name="left_camera_joint" type="fixed">
+    <parent link="base_link"/>
+    <child link="left_camera_link"/>
+    <origin xyz="0.7 -0.63 0.5" rpy="0 0.05 -1.0"/>
+  </joint>
+  <link name="left_camera_link_optical">
+    <inertial>
+      <mass value="1" />
+      <inertia ixx="0.001" ixy="0.0" ixz="0.0" iyy="0.001" iyz="0.0" izz="0.001"/>
+    </inertial>
+  </link>
+  <joint name="left_camera_optical_joint" type="fixed">
+    <origin xyz="0 0 0" rpy="-1.5707 0 -1.5707"/>
+    <parent link="left_camera_link"/>
+    <child link="left_camera_link_optical"/>
+  </joint>
+  <!-- right camera -->
+  <link name="right_camera_link">
+    <inertial>
+      <mass value="1"/>
+      <inertia ixx="0.001" ixy="0.0" ixz="0.0" iyy="0.001" iyz="0.0" izz="0.001"/>
+    </inertial>
+    <visual>
+      <origin xyz="0 0 0" rpy="0 0 0"/>
+      <geometry>
+        <box size="0.010 0.03 0.03"/>
+      </geometry>
+      <material name="red"/>
+    </visual>
+  </link>
+  <joint name="right_camera_joint" type="fixed">
+    <parent link="base_link"/>
+    <child link="right_camera_link"/>
+    <origin xyz="-0.7 -0.63 0.5" rpy="0 0.05 -2.1416"/>
+  </joint>
+  <link name="right_camera_link_optical">
+    <inertial>
+      <mass value="1"/>
+      <inertia ixx="0.001" ixy="0.0" ixz="0.0" iyy="0.001" iyz="0.0" izz="0.001"/>
+    </inertial>
+  </link>
+  <joint name="right_camera_optical_joint" type="fixed">
+    <origin xyz="0 0 0" rpy="-1.5707 0 -1.5707"/>
+    <parent link="right_camera_link"/>
+    <child link="right_camera_link_optical"/>
+  </joint>
+  <!-- Gazebo refs -->
+  <gazebo reference="front_camera_link">
+    <material>Gazebo/Red</material>
+    <sensor type="camera" name="front_camera_sensor">
+      <update_rate>30.0</update_rate>
+      <pose>0 0 0 0 0 0</pose>
+      <visualize>true</visualize>
+      <camera name="front_camera">
+        <horizontal_fov>1.3962634</horizontal_fov>
+        <image>
+          <width>800</width>
+          <height>800</height>
+          <format>R8G8B8</format>
+        </image>
+        <clip>
+          <near>0.02</near>
+          <far>300</far>
+        </clip>
+      </camera>
+      <plugin name="front_camera_controller" filename="libgazebo_ros_camera.so">
+        <imageTopicName>image_raw</imageTopicName>
+        <topic_name>/prius/front_camera</topic_name>
+        <frame_name>front_camera_link_optical</frame_name>
+        <min_depth>0.02</min_depth>
+        <max_depth>300.0</max_depth>
+      </plugin>
+    </sensor>
+  </gazebo>
+  <gazebo reference="back_camera_link">
+    <material>Gazebo/Red</material>
+    <sensor type="camera" name="back_camera_sensor">
+      <update_rate>30.0</update_rate>
+      <pose>0 0 0 0 0 0</pose>
+      <visualize>false</visualize>
+      <camera name="back_camera">
+        <horizontal_fov>1.3962634</horizontal_fov>
+        <image>
+          <width>800</width>
+          <height>800</height>
+          <format>R8G8B8</format>
+        </image>
+        <clip>
+          <near>0.02</near>
+          <far>300</far>
+        </clip>
+      </camera>
+      <plugin name="back_camera_controller" filename="libgazebo_ros_camera.so">
+        <imageTopicName>image_raw</imageTopicName>
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
Commit message: fixed Lidar

File: car_ws/src/auto_park2/description/prius.urdf.xacro (robot description, xacro)
@@ -119,9 +119,10 @@
     </inertial>
   </link>
-  <joint name="front_left_steer_joint" type="fixed">
+  <joint name="front_left_steer_joint" type="revolute">
     <parent link="base_link"/>
     <child link="fl_axle"/>
     <origin xyz="0.8 0 0" rpy="0 0 0"/>
     <axis xyz="0 0 1"/>
+    <limit effort="100.0" velocity="10.0" lower="-0.8727" upper="0.8727"/>
   </joint>
   <!-- front right_wheel -->
@@ -159,9 +160,10 @@
     </inertial>
   </link>
-  <joint name="front_right_steer_joint" type="fixed">
+  <joint name="front_right_steer_joint" type="revolute">
     <parent link="base_link"/>
     <child link="fr_axle"/>
     <origin xyz="-0.8 0 0" rpy="0 0 0"/>
     <axis xyz="0 0 1"/>
+    <limit effort="100.0" velocity="10.0" lower="-0.8727" upper="0.8727"/>
   </joint>
   <!-- rear left_wheel -->
@@ -230,7 +232,7 @@
   </link>
   <joint name="scan_joint" type="fixed">
-    <parent link="base_link"/>
+    <parent link="front_camera_link"/>
     <child link="base_scan"/>
-    <origin xyz="0 0.5 1.125" rpy="0 0 -1.5707"/>
+    <origin xyz="0.53 0.0 -0.3" rpy="0 0 0"/>
   </joint>
   <!-- front camera -->
@@ -475,6 +477,6 @@
             <samples>360</samples>
             <resolution>1</resolution>
-            <min_angle>-1.8</min_angle>
-            <max_angle>1.8</max_angle>
+            <min_angle>-1.72</min_angle>
+            <max_angle>1.72</max_angle>
           </horizontal>
         </scan>
@@ -537,4 +539,22 @@
       <state_interface name="position"/>
     </joint>
+    <joint name="front_left_steer_joint">
+      <command_interface name="position">
+        <param name="min">-0.8727</param>
+        <param name="max">0.8727</param>
+      </command_interface>
+      <state_interface name="velocity"/>
+      <state_interface name="position"/>
+      <state_interface name="effort" />
+    </joint>
+    <joint name="front_right_steer_joint">
+      <command_interface name="position">
+        <param name="min">-0.8727</param>
+        <param name="max">0.8727</param>
+      </command_interface>
+      <state_interface name="velocity"/>
+      <state_interface name="position"/>
+      <state_interface name="effort" />
+    </joint>
   </ros2_control>
   <gazebo>

Commit message: car mostly done

File: car_ws/src/auto_park2/description/prius.urdf.xacro (robot description, xacro)
@@ -19,5 +19,5 @@
       <origin xyz="0 1.42 -0.3" rpy="0 0 0"/>
       <geometry>
-        <mesh filename="file:///home/andrew/auto_parking/car_ws/src/auto_park2/description/hybrid_body.obj" scale="0.01 0.01 0.01"/>
+        <mesh filename="file:///home/ubuntu/auto_parking/car_ws/src/auto_park2/description/hybrid_body.obj" scale="0.01 0.01 0.01"/>
       </geometry>
       <material name="light_black"/>
@@ -26,5 +26,5 @@
       <origin xyz="0.0 0.05 0.625" rpy="0 0 0"/>
       <geometry>
-        <box size="1.7526 2.1 0.95"/>
+        <box size="1 0.9 0.75"/>
       </geometry>
     </collision>
@@ -32,5 +32,5 @@
       <origin xyz="0.0 -2.0 0.458488" rpy="0.0 0 0"/>
       <geometry>
-        <box size="1.337282 0.48 0.566691"/>
+        <box size="0.337282 0.28 0.266691"/>
       </geometry>
     </collision>
@@ -38,5 +38,5 @@
       <origin xyz="0.0 -1.900842 0.676305" rpy="0.341247 0 0"/>
       <geometry>
-        <box size="1.597968 0.493107 0.265468"/>
+        <box size="0.397968 0.293107 0.165468"/>
       </geometry>
     </collision>
@@ -44,5 +44,5 @@
       <origin xyz="0.0 -0.875105 1.032268" rpy="0.335476 0 0"/>
       <geometry>
-        <box size="1.168381 1.654253 0.272347"/>
+        <box size="0.168381 0.654253 0.272347"/>
       </geometry>
     </collision>
@@ -50,5 +50,5 @@
       <origin xyz="0.0 0.161236 1.386042" rpy="0.135030 0 0"/>
       <geometry>
-        <box size="1.279154 0.625988 0.171868"/>
+        <box size="0.279154 0.625988 0.171868"/>
       </geometry>
     </collision>
@@ -56,5 +56,5 @@
       <origin xyz="0.0 0.817696 1.360069" rpy="-0.068997 0 0"/>
       <geometry>
-        <box size="1.285130 0.771189 0.226557"/>
+        <box size="0.285130 0.771189 0.226557"/>
       </geometry>
     </collision>
@@ -62,5 +62,5 @@
       <origin xyz="0.0 1.640531 1.175126" rpy="-0.262017 0 0"/>
       <geometry>
-        <box size="1.267845 1.116344 0.244286"/>
+        <box size="0.267845 0.116344 0.244286"/>
       </geometry>
     </collision>
@@ -68,5 +68,5 @@
       <origin xyz="0.0 1.637059 0.888180" rpy="0.0 0 0"/>
       <geometry>
-        <box size="1.788064 1.138988 0.482746"/>
+        <box size="0.788064 0.138988 0.482746"/>
       </geometry>
     </collision>
@@ -74,5 +74,5 @@
       <origin xyz="0.0 2.054454 0.577870" rpy="0.0 0 0"/>
       <geometry>
-        <box size="1.781650 0.512093 0.581427"/>
+        <box size="0.781650 0.512093 0.581427"/>
       </geometry>
     </collision>
@@ -97,5 +97,5 @@
       <origin xyz="0 0 0" rpy="0 0 0"/>
       <geometry>
-        <mesh filename="file:///home/andrew/auto_parking/car_ws/src/auto_park2/description/wheel.obj" scale="0.01 0.01 0.01"/>
+        <mesh filename="file:///home/ubuntu/auto_parking/car_ws/src/auto_park2/description/wheel.obj" scale="0.01 0.01 0.01"/>
       </geometry>
     </visual>
@@ -138,5 +138,5 @@
       <origin xyz="0 0 0" rpy="0 0 0"/>
       <geometry>
-        <mesh filename="file:///home/andrew/auto_parking/car_ws/src/auto_park2/description/wheel.obj" scale="0.01 0.01 0.01"/>
+        <mesh filename="file:///home/ubuntu/auto_parking/car_ws/src/auto_park2/description/wheel.obj" scale="0.01 0.01 0.01"/>
       </geometry>
     </visual>
@@ -178,5 +178,5 @@
       <origin xyz="0 0 0" rpy="0 0 0"/>
       <geometry>
-        <mesh filename="file:///home/andrew/auto_parking/car_ws/src/auto_park2/description/wheel.obj" scale="0.01 0.01 0.01"/>
+        <mesh filename="file:///home/ubuntu/auto_parking/car_ws/src/auto_park2/description/wheel.obj" scale="0.01 0.01 0.01"/>
       </geometry>
     </visual>
@@ -203,5 +203,5 @@
       <origin xyz="0 0 0" rpy="0 0 0"/>
       <geometry>
-        <mesh filename="file:///home/andrew/auto_parking/car_ws/src/auto_park2/description/wheel.obj" scale="0.01 0.01 0.01"/>
+        <mesh filename="file:///home/ubuntu/auto_parking/car_ws/src/auto_park2/description/wheel.obj" scale="0.01 0.01 0.01"/>
       </geometry>
     </visual>
@@ -313,5 +313,5 @@
     <parent link="base_link"/>
     <child link="left_camera_link"/>
-    <origin xyz="0.7 -0.63 0.5" rpy="0 0.05 -1.0"/>
+    <origin xyz="0.7 -0.63 0.5" rpy="0 0.05 -0.65"/>
   </joint>
   <link name="left_camera_link_optical">
@@ -343,5 +343,5 @@
     <parent link="base_link"/>
     <child link="right_camera_link"/>
-    <origin xyz="-0.7 -0.63 0.5" rpy="0 0.05 -2.1416"/>
+    <origin xyz="-0.7 -0.63 0.5" rpy="0 0.05 -2.4916"/>
   </joint>
   <link name="right_camera_link_optical">
@@ -362,5 +362,5 @@
       <update_rate>30.0</update_rate>
       <pose>0 0 0 0 0 0</pose>
-      <visualize>true</visualize>
+      <visualize>false</visualize>
       <camera name="front_camera">
         <horizontal_fov>1.3962634</horizontal_fov>
@@ -470,5 +470,5 @@
     <sensor type="ray" name="lds_lfcd_sensor">
       <pose>0 0 0 0 0 0</pose>
-      <visualize>true</visualize>
+      <visualize>false</visualize>
       <update_rate>10</update_rate>
       <ray>
@@ -560,5 +560,5 @@
   <gazebo>
     <plugin name="gazebo_ros2_control" filename="libgazebo_ros2_control.so">
-      <parameters>/home/andrew/auto_parking/car_ws/src/auto_park2/config/controllers.yaml</parameters>
+      <parameters>/home/ubuntu/auto_parking/car_ws/src/auto_park2/config/controllers.yaml</parameters>
       <odometry_frame>odom</odometry_frame>
       <robot_base_frame>base_link</robot_base_frame>

Commit message: fix collision

File: car_ws/src/auto_park2/description/prius.urdf.xacro (robot description, xacro)
@@ -26,23 +26,11 @@
       <origin xyz="0.0 0.05 0.625" rpy="0 0 0"/>
       <geometry>
-        <box size="1 0.9 0.75"/>
-      </geometry>
-    </collision>
-    <collision name="front_bumper">
-      <origin xyz="0.0 -2.0 0.458488" rpy="0.0 0 0"/>
-      <geometry>
-        <box size="0.337282 0.28 0.266691"/>
-      </geometry>
-    </collision>
-    <collision name="hood">
-      <origin xyz="0.0 -1.900842 0.676305" rpy="0.341247 0 0"/>
-      <geometry>
-        <box size="0.397968 0.293107 0.165468"/>
+        <box size="1.4 1.2 0.75"/>
       </geometry>
     </collision>
     <collision name="windshield">
-      <origin xyz="0.0 -0.875105 1.032268" rpy="0.335476 0 0"/>
-      <geometry>
-        <box size="0.168381 0.654253 0.272347"/>
+      <origin xyz="0.0 0 1.032268" rpy="0.335476 0 0"/>
+      <geometry>
+        <box size="0.168381 0.354253 0.272347"/>
       </geometry>
     </collision>

Commit message: added Joint trajectory controller

File: car_ws/src/auto_park2/description/prius.urdf.xacro (robot description, xacro)
@@ -112,5 +112,5 @@
     <origin xyz="0.8 0 0" rpy="0 0 0"/>
     <axis xyz="0 0 1"/>
-    <limit effort="100.0" velocity="10.0" lower="-0.8727" upper="0.8727"/>
+    <limit effort="100.0" velocity="10.0" lower="-0.8728" upper="0.8728"/>
   </joint>
   <!-- front right_wheel -->
@@ -153,5 +153,5 @@
     <origin xyz="-0.8 0 0" rpy="0 0 0"/>
     <axis xyz="0 0 1"/>
-    <limit effort="100.0" velocity="10.0" lower="-0.8727" upper="0.8727"/>
+    <limit effort="100.0" velocity="10.0" lower="-0.8728" upper="0.8728"/>
   </joint>
   <!-- rear left_wheel -->
