Commit message: Added Lidar functionality, reformatted launch files

File: car_ws/src/auto_park2/description/prius.urdf.xacro (robot description, xacro)
@@ -24,7 +24,7 @@
     </visual>
     <collision name="chassis">
-      <origin xyz="0.0 0.05 0.625" rpy="0 0 0"/>
-      <geometry>
-        <box size="1.4 1.2 0.75"/>
+      <origin xyz="0.0 0.05 0.425" rpy="0 0 0"/>
+      <geometry>
+        <box size="1.4 1.4 0.35"/>
       </geometry>
     </collision>
@@ -222,5 +222,5 @@
     <parent link="front_camera_link"/>
     <child link="base_scan"/>
-    <origin xyz="0.53 0.0 -0.3" rpy="0 0 0"/>
+    <origin xyz="0.13 0.0 0.3" rpy="0 0 0"/>
   </joint>
   <!-- front camera -->
@@ -458,5 +458,5 @@
     <sensor type="ray" name="lds_lfcd_sensor">
       <pose>0 0 0 0 0 0</pose>
-      <visualize>false</visualize>
+      <visualize>true</visualize>
       <update_rate>10</update_rate>
       <ray>
@@ -465,6 +465,6 @@
             <samples>360</samples>
             <resolution>1</resolution>
-            <min_angle>-1.72</min_angle>
-            <max_angle>1.72</max_angle>
+            <min_angle>-2.0</min_angle>
+            <max_angle>2.0</max_angle>
           </horizontal>
         </scan>
